File: KiCad/robotics_20240527/robotics_20240527.kicad_pcb (KiCad board)
At the start: 2 copper layers, 18 parts, among them IC1 BNO085, U1 MPU-6050, U2 LD1117S50TR_SOT223, U5 MPU-6050

Commit message: add_stm_1
Parts:
- removed C6: 0.1uC, Capacitor_SMD:C_0603_1608Metric_Pad1.08x0.95mm_HandSolder
- removed R3: 1kR, Resistor_SMD:R_0603_1608Metric_Pad0.98x0.95mm_HandSolder
- added BA1: ~, Connector_JST:JST_PH_B2B-PH-K_1x02_P2.00mm_Vertical, B.Cu at (215.7, 59.0)
- added C10: 0.1uC, Capacitor_SMD:C_0603_1608Metric_Pad1.08x0.95mm_HandSolder, F.Cu at (200.5, 79.2)
- added C11: 22pC, Capacitor_SMD:C_0603_1608Metric_Pad1.08x0.95mm_HandSolder, F.Cu at (196.0, 74.2)
- added C12: 22pC, Capacitor_SMD:C_0603_1608Metric_Pad1.08x0.95mm_HandSolder, F.Cu at (196.0, 70.6)
- added C13: 4.7uC, Capacitor_SMD:C_0603_1608Metric_Pad1.08x0.95mm_HandSolder, F.Cu at (195.0, 57.2)
- added C14: 0.1uC, Capacitor_SMD:C_0603_1608Metric_Pad1.08x0.95mm_HandSolder, F.Cu at (182.9, 74.2)
- added C15: 0.1uC, Capacitor_SMD:C_0603_1608Metric_Pad1.08x0.95mm_HandSolder, F.Cu at (189.6, 74.2)
- added C19: 0.1uC, Capacitor_SMD:C_0603_1608Metric_Pad1.08x0.95mm_HandSolder, F.Cu at (175.8, 68.6)
- added C20: 0.1uC, Capacitor_SMD:C_0603_1608Metric_Pad1.08x0.95mm_HandSolder, F.Cu at (175.8, 70.7)
- added C21: 0.1uC, Capacitor_SMD:C_0603_1608Metric_Pad1.08x0.95mm_HandSolder, F.Cu at (175.8, 63.6)
- added C24: 4.7uC, Capacitor_SMD:C_0603_1608Metric_Pad1.08x0.95mm_HandSolder, F.Cu at (190.5, 76.8)
- added C8: 0.1uC, Capacitor_SMD:C_0603_1608Metric_Pad1.08x0.95mm_HandSolder, F.Cu at (211.5, 74.1)
- added C9: 0.1uC, Capacitor_SMD:C_0603_1608Metric_Pad1.08x0.95mm_HandSolder, F.Cu at (200.5, 76.9)
- added D2: IR26, LED_SMD:LED_1206_3216Metric, F.Cu at (205.9, 88.8)
- added D3: IR26, LED_SMD:LED_1206_3216Metric, F.Cu at (197.3, 88.9)
- added D4: IR26, LED_SMD:LED_1206_3216Metric, F.Cu at (199.9, 88.9)
- added M1: ~, Connector_JST:JST_PH_B2B-PH-K_1x02_P2.00mm_Vertical, B.Cu at (170.9, 43.5)
- added M2: ~, Connector_JST:JST_PH_B2B-PH-K_1x02_P2.00mm_Vertical, B.Cu at (213.4, 45.3)
- added M3: ~, Connector_JST:JST_PH_B2B-PH-K_1x02_P2.00mm_Vertical, B.Cu at (211.5, 86.4)
- added M4: ~, Connector_JST:JST_PH_B2B-PH-K_1x02_P2.00mm_Vertical, B.Cu at (169.8, 85.3)
- added R10: 10kR, Resistor_SMD:R_0603_1608Metric_Pad0.98x0.95mm_HandSolder, B.Cu at (189.4, 42.7)
- added R11: 10kR, Resistor_SMD:R_0603_1608Metric_Pad0.98x0.95mm_HandSolder, B.Cu at (189.5, 86.4)
- added R12: 10kR, Resistor_SMD:R_0603_1608Metric_Pad0.98x0.95mm_HandSolder, B.Cu at (189.5, 89.9)
- added R13: R, Resistor_SMD:R_0603_1608Metric_Pad0.98x0.95mm_HandSolder, B.Cu at (192.0, 90.8)
- added R14: R, Resistor_SMD:R_0603_1608Metric_Pad0.98x0.95mm_HandSolder, B.Cu at (186.8, 41.8)
- added R15: R, Resistor_SMD:R_0603_1608Metric_Pad0.98x0.95mm_HandSolder, B.Cu at (186.8, 45.4)
- added R16: 1kR, Resistor_SMD:R_0603_1608Metric_Pad0.98x0.95mm_HandSolder, F.Cu at (197.3, 84.6)
- added R17: 1kR, Resistor_SMD:R_0603_1608Metric_Pad0.98x0.95mm_HandSolder, F.Cu at (199.9, 84.5)
- added R18: 1kR, Resistor_SMD:R_0603_1608Metric_Pad0.98x0.95mm_HandSolder, F.Cu at (203.4, 84.7)
- added R19: 1kR, Resistor_SMD:R_0603_1608Metric_Pad0.98x0.95mm_HandSolder, F.Cu at (205.9, 84.7)
- added R4: 10kR, Resistor_SMD:R_0603_1608Metric_Pad0.98x0.95mm_HandSolder, F.Cu at (209.1, 78.4)
- added R5: R, Resistor_SMD:R_0603_1608Metric_Pad0.98x0.95mm_HandSolder, B.Cu at (192.1, 87.3)
- added R6: 10kR, Resistor_SMD:R_0603_1608Metric_Pad0.98x0.95mm_HandSolder, F.Cu at (205.5, 78.4)
- added R7: 10kR, Resistor_SMD:R_0603_1608Metric_Pad0.98x0.95mm_HandSolder, F.Cu at (207.3, 78.4)
- added R8: 10kR, Resistor_SMD:R_0603_1608Metric_Pad0.98x0.95mm_HandSolder, F.Cu at (181.4, 52.0)
- added R9: 10kR, Resistor_SMD:R_0603_1608Metric_Pad0.98x0.95mm_HandSolder, B.Cu at (189.4, 46.3)
- added ST-Link1: ~, Connector_JST:JST_PH_S6B-PH-K_1x06_P2.00mm_Horizontal, B.Cu at (171.3, 74.5)
- added U3: STM32F446RETx, Package_QFP:LQFP-64_10x10mm_P0.5mm, F.Cu at (185.8, 64.3)
- added U4: μPA2753GR, Package_SO:HSOP-8-1EP_3.9x4.9mm_P1.27mm_EP2.3x2.3mm, B.Cu at (194.8, 44.3)
- added UART1: ~, Connector_JST:JST_PH_B2B-PH-K_1x02_P2.00mm_Vertical, B.Cu at (168.2, 57.2)
- added Y1: 32.768KHZ, Crystal:Crystal_SMD_MicroCrystal_CC7V-T1A-2Pin_3.2x1.5mm_HandSoldering, F.Cu at (199.1, 72.4)
- C16: value 10nC -> 0.1uC
- C17, C18: value 0.1µC -> 0.1uC
- C5: value 4.7uC -> 10uC; moved to B.Cu
- C7: value 10nC -> 10uC; moved to B.Cu
- D1: value IR26-21C_L110_TR8 -> IR26
- U2: moved to B.Cu
- U5: value MPU-6050 -> μPA2753GR; footprint Sensor_Motion:InvenSense_QFN-24_4x4mm_P0.5mm -> Package_SO:HSOP-8-1EP_3.9x4.9mm_P1.27mm_EP2.3x2.3mm; moved to B.Cu
- moved C3 165.6 mm to (216.3, 66.6), turned to 0 degrees
- moved C1 161.6 mm to (216.3, 68.8), turned to 0 degrees
- moved U1 161.3 mm to (211.3, 68.1)
- moved C2 160.5 mm to (211.2, 64.3)
- moved C4 160.1 mm to (207.5, 66.5)
- moved D1 155.0 mm to (203.3, 88.8), turned to 90 degrees
- moved C16 151.1 mm to (195.0, 59.0), turned to 180 degrees
- moved U5 149.3 mm to (183.9, 87.9)
- moved R2 146.2 mm to (199.8, 66.8), turned to 180 degrees
- moved C7 144.6 mm to (207.0, 55.2)
- moved R1 143.1 mm to (198.6, 65.2), turned to 180 degrees
- moved IC1 141.7 mm to (204.7, 72.4), turned to 180 degrees
- moved C17 139.4 mm to (180.6, 56.1), turned to -90 degrees
- moved C5 136.3 mm to (209.2, 57.3), turned to 90 degrees
- moved C18 136.2 mm to (175.8, 66.6), turned to 0 degrees
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Connections:
- net +5V renamed +3.7V
- C1 pad 1: +3.3V -> STL-1
- C1 pad 2: GND -> STL-2
- C16 pad 1: +3.3V -> STL-2
- C16 pad 2: GND -> STL-1
- C17 pad 1: +3.3V -> STL-2
- C17 pad 2: GND -> STL-1
- C18 pad 1: Net-(U5-REGOUT) -> STL-2
- C18 pad 2: GND -> STL-1
- C2 pad 1: +3.3V -> STL-1
- C2 pad 2: GND -> STL-2
- C3 pad 2: GND -> STL-2
- C4 pad 2: GND -> STL-2
- C5 pad 2: GND -> STL-2
- C7 pad 1: +3.3V -> STL-1
- C7 pad 2: GND -> STL-2
- D1 pad 1: GND -> STL-2
- IC1 pad 10: unconnected-(IC1-CLKSEL0-Pad10) -> CLKSEL
- IC1 pad 11: unconnected-(IC1-NRST-Pad11) -> RST
- IC1 pad 14: unconnected-(IC1-H_INTN-Pad14) -> INT
- IC1 pad 19: unconnected-(IC1-H_SCL/SCK/RX-Pad19) -> SCL
- IC1 pad 2: unconnected-(IC1-GND_1-Pad2) -> STL-2
- IC1 pad 20: unconnected-(IC1-H_SDA/H_MISO/TX_-Pad20) -> SDA
- IC1 pad 25: unconnected-(IC1-GND_2-Pad25) -> STL-2
- IC1 pad 26: unconnected-(IC1-XOUT32/CLKSEL1-Pad26) -> Net-(IC1-XOUT32/CLKSEL1)
- IC1 pad 27: unconnected-(IC1-XIN32-Pad27) -> Net-(IC1-XIN32)
- IC1 pad 28: unconnected-(IC1-VDDIO-Pad28) -> STL-1
- IC1 pad 3: unconnected-(IC1-VDD-Pad3) -> STL-1
- IC1 pad 4: unconnected-(IC1-BOOTN-Pad4) -> BOOTN
- IC1 pad 5: unconnected-(IC1-PS1-Pad5) -> STL-2
- IC1 pad 6: unconnected-(IC1-PS0/WAKE-Pad6) -> STL-2
- IC1 pad 9: unconnected-(IC1-CAP-Pad9) -> Net-(IC1-CAP)
- R1 pad 1: +3.3V -> STL-1
- R2 pad 1: +3.3V -> STL-1
- U1 pad 1: GND -> STL-2
- U1 pad 11: GND -> STL-2
- U1 pad 13: +3.3V -> STL-1
- U1 pad 18: GND -> STL-2
- U1 pad 8: +3.3V -> STL-1
- U1 pad 9: AD0 -> unconnected-(U1-AD0-Pad9)
- U2 pad 1: GND -> STL-2
- U2 pad 2: +3.3V -> STL-1
- U5 pad 1: GND -> STL-2
- U5 pad 2: unconnected-(U5-NC-Pad2) -> Net-(U5-G1)
- U5 pad 3: unconnected-(U5-NC-Pad3) -> STL-2
- U5 pad 4: unconnected-(U5-NC-Pad4) -> Net-(U5-G2)
- U5 pad 5: unconnected-(U5-NC-Pad5) -> M4
- U5 pad 6: unconnected-(U5-AUX_DA-Pad6) -> M4
- U5 pad 7: unconnected-(U5-AUX_CL-Pad7) -> M3
- U5 pad 8: +3.3V -> M3
Routing:
- net STL-2: track 0.00 -> 478.7 mm, vias 0 -> 193
- net STL-1: track 0.00 -> 207.4 mm, vias 0 -> 17
- net +3.7V: track 7.15 -> 169.7 mm
- net GND: track 161.1 -> 0.00 mm, vias 5 -> 0
- net CLKSEL: track 0.00 -> 55.0 mm, vias 0 -> 2
- net STL-4: track 0.00 -> 50.5 mm, vias 0 -> 1
- net RST: track 0.00 -> 48.0 mm, vias 0 -> 2
- net INT: track 0.00 -> 45.5 mm, vias 0 -> 2
- net M4G2: track 0.00 -> 41.1 mm, vias 0 -> 1
- net M3: track 0.00 -> 39.8 mm
- net M1: track 0.00 -> 38.1 mm
- net M3G1: track 0.00 -> 38.0 mm, vias 0 -> 1
- net +3.3V: track 37.4 -> 0.00 mm, vias 3 -> 0
- net STL-5: track 0.00 -> 36.9 mm, vias 0 -> 1
- net BOOTN: track 0.00 -> 31.3 mm, vias 0 -> 2
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- added copper zone on B.Cu, net STL-2
- added copper zone on F.Cu, net STL-2
Other:
- board outline added: 88 x 88 mm
- board text added: "- +"
- board text added: "3.7v"
- board text added: "6 5 4 3"
- board text added: "GND 3.3"
- board text added: "M"
- board text added: "TX RX"
