File: KiCad/robotics_20240527/robotics_20240527.kicad_sch (KiCad schematic)
At the start: 23 parts, among them IC1 BNO085, U1 MPU-6050, U2 LD1117S50TR_SOT223, U5 MPU-6050

Commit message: add_stm_1
Parts:
- removed C6: 0.1uC, Capacitor_SMD:C_0603_1608Metric_Pad1.08x0.95mm_HandSolder, symbol Device:C
- removed R3: 1kR, Resistor_SMD:R_0603_1608Metric_Pad0.98x0.95mm_HandSolder, symbol Device:R
- removed U5: MPU-6050, Sensor_Motion:InvenSense_QFN-24_4x4mm_P0.5mm, symbol Sensor_Motion:MPU-6050
- added BA1, M1, M2, M3, M4, UART1: ~, Connector_JST:JST_PH_B2B-PH-K_1x02_P2.00mm_Vertical, symbol XH_01x02:XH_01_02
- added C11, C12: 22pC, Capacitor_SMD:C_0603_1608Metric_Pad1.08x0.95mm_HandSolder, symbol Device:C
- added C13, C24: 4.7uC, Capacitor_SMD:C_0603_1608Metric_Pad1.08x0.95mm_HandSolder, symbol Device:C
- added C14, C15, C20, C21: 0.1uC, Capacitor_SMD:C_0603_1608Metric_Pad1.08x0.95mm_HandSolder, symbol Device:C
- added D2, D3, D4: IR26, LED_SMD:LED_1206_3216Metric, symbol LED:IR26-21C_L110_TR8
- added R10, R11, R12, R6, R7, R8, R9: 10kR, Resistor_SMD:R_0603_1608Metric_Pad0.98x0.95mm_HandSolder, symbol Device:R
- added R13, R14, R15, R5: R, Resistor_SMD:R_0603_1608Metric_Pad0.98x0.95mm_HandSolder, symbol Device:R
- added R16, R17, R18, R19: 1kR, Resistor_SMD:R_0603_1608Metric_Pad0.98x0.95mm_HandSolder, symbol Device:R
- added ST-Link1: ~, Connector_JST:JST_PH_S6B-PH-K_1x06_P2.00mm_Horizontal, symbol XH_01x06:XH_01x06
- added U3: STM32F446RETx, Package_QFP:LQFP-64_10x10mm_P0.5mm, symbol MCU_ST_STM32F4:STM32F446RETx
- added U4, U5: μPA2753GR, Package_SO:HSOP-8-1EP_3.9x4.9mm_P1.27mm_EP2.3x2.3mm, symbol μPA2753GR:μPA2753GR
- added Y1: 32.768KHZ, Crystal:Crystal_SMD_MicroCrystal_CC7V-T1A-2Pin_3.2x1.5mm_HandSoldering, symbol Device:Crystal
- C10, C8, C9: footprint (none) -> Capacitor_SMD:C_0603_1608Metric_Pad1.08x0.95mm_HandSolder
- C16: value 10nC -> 0.1uC
- C17, C18: value 0.1µC -> 0.1uC
- C19: value 2.2nC -> 0.1uC
- C5: value 4.7uC -> 10uC
- C7: value 10nC -> 10uC
- D1: value IR26-21C_L110_TR8 -> IR26
- R4: footprint (none) -> Resistor_SMD:R_0603_1608Metric_Pad0.98x0.95mm_HandSolder
Connections:
- net +3.3V: now also C16.2, C17.2, C18.2, C19.2, C13.1, C14.2, C15.2, C20.2, R6.1, R7.1, ST-Link1.1, U3.1 (VBAT), U3.13 (VDDA), U3.19 (VDD), U3.32 (VDD), U3.48 (VDD), U3.64 (VDD); no longer C16.1, C17.1
- net GND: now also C16.1, C17.1, C18.1, C19.1, IC1.2 (GND_1), IC1.25 (GND_2), IC1.5 (PS1), IC1.6 (PS0/WAKE), BA1.2, C11.1, C12.1, C13.2, C14.1, C15.1, C20.1, C21.2, C24.2, D2.1 (K), D3.1 (K), D4.1 (K), R10.1, R11.1, R12.1, R8.2, R9.1, ST-Link1.2, U3.12 (VSSA), U3.18 (VSS), U3.31 (VSS), U3.47 (VSS), U3.63 (VSS), U4.1 (S1), U4.3 (S2), U5.1 (S1), U5.3 (S2); no longer C16.2, C17.2, C18.2, C19.2
- net RST: now also U3.58 (PB6)
- net SCL: now also IC1.19 (H_SCL/SCK/RX), U3.37 (PC6)
- net SDA: now also IC1.20 (H_SDA/H_MISO/TX_), U3.38 (PC7)
- net at D1.2 (A): now also R18.1
- net CLKSEL: now reaches IC1.10 (CLKSEL0)
- net CLKSEL: now also R7.2, U3.61 (PB8)
- net INT: now reaches IC1.14 (H_INTN)
- net INT: now also U3.62 (PB9)
- net at IC1.26 (XOUT32/CLKSEL1): now also C12.2, Y1.2
- net at IC1.27 (XIN32): now also C11.2, Y1.1
- net BOOTN: now reaches IC1.4 (BOOTN)
- net BOOTN: now also R6.2, U3.29 (PB10)
- net +5V renamed +3.7V
- net +3.7V: now also BA1.1, M1.1, M2.1, M3.1, M4.1
- net AD0: no longer names the net of U1.9 (AD0)
- new net: D3.2 (A), R16.1
- new net: R16.2, U3.21 (PA5)
- new net: R12.2, R13.2, U5.4 (G2)
- new net: D2.2 (A), R19.1
- new net: R15.2, R9.2, U4.2 (G1)
- new net: R10.2, R14.2, U4.4 (G2)
- new net: R8.1, U3.60 (BOOT0)
- new net: R17.2, U3.23 (PA7)
- new net: C24.1, U3.30 (VCAP_1)
- new net: R18.2, U3.34 (PB13)
- new net: R19.2, U3.36 (PB15)
- new net: D4.2 (A), R17.1
- new net: R11.2, R5.2, U5.2 (G1)
- new net M1: M1.2, U4.7 (D1), U4.8 (D1)
- new net M1G1: R15.1, U3.57 (PB5)
- new net M2: M2.2, U4.5 (D2), U4.6 (D2)
- new net M2G2: R14.1, U3.59 (PB7)
- new net M3: M3.2, U5.7 (D1), U5.8 (D1)
- new net M3G1: R5.1, U3.14 (PA0)
- new net M4: M4.2, U5.5 (D2), U5.6 (D2)
- new net M4G2: R13.1, U3.15 (PA1)
- new net RX: U3.52 (PC11), UART1.2
- new net STL-3: C21.1, ST-Link1.3, U3.7 (NRST)
- new net STL-4: ST-Link1.4, U3.49 (PA14)
- new net STL-5: ST-Link1.5, U3.46 (PA13)
- new net STL-6: ST-Link1.6, U3.55 (PB3)
- new net TX: U3.51 (PC10), UART1.1
- no-connect marks 6 -> 48
Other:
- moved on the sheet: C1, C10, C2, C3, C4, C5, C7, C8, C9, IC1, R1, R2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
